Commit message: Friction and camera position

File: franka_description/robots/panda.gazebo.xacro (robot description, xacro)
@@ -65,12 +65,18 @@
         <gazebo reference="${robot_name}_rightfinger">
             <material>Gazebo/Grey</material>
-            <mu1>0.2</mu1>
-            <mu2>0.2</mu2>
+	    <kp>1000000</kp>
+	    <kd>1.0</kd>
+            <mu1>1.0</mu1>
+            <mu2>1.0</mu2>
+	    <minDepth>0.001</minDepth>
         </gazebo>
         <!-- LinkLeftFinger -->
         <gazebo reference="${robot_name}_leftfinger">
             <material>Gazebo/Grey</material>
-            <mu1>0.2</mu1>
-            <mu2>0.2</mu2>
+	    <kp>1000000</kp>
+	    <kd>1.0</kd>
+            <mu1>100.0</mu1>
+            <mu2>100.0</mu2>
+	    <minDepth>0.001</minDepth>
         </gazebo>
     </xacro:macro>

File: franka_description/robots/panda_arm.xacro (robot description, xacro)
@@ -11,5 +11,5 @@
     <!-- for simulation -->
     <link name="world" />
-    <joint name="robot_to_world" type="fixed">
+    <joint name="virtual_joint" type="fixed">
       <parent link="world" />
       <child link="${arm_id}_link0" />

File: franka_description/robots/panda_arm_hand.urdf.xacro (robot description, xacro)
@@ -14,8 +14,10 @@
   <xacro:panda_transmission robot_name="$(arg robot_name)" load_hand="true" />
   <!-- end for simulation -->
-<!--Camera link and plugin-->
-   <xacro:include filename="$(find realsense_gazebo_plugin)/urdf/realsense-RS200.macro.xacro"/>
-   <xacro:realsense-rs200 prefix="" parent="panda_link8">
-        <origin xyz="0.05 0 0.05" rpy="${-pi/4} ${-pi/2} 0" />
-   </xacro:realsense-rs200>
+  <!--Camera link plugin-->
+  <xacro:include filename="$(find realsense_gazebo_plugin)/urdf/realsense-RS200.macro.xacro"/>
+  <xacro:realsense-rs200 prefix="" parent="panda_link8">
+       <!--Position of the camera wrt to link 8 -->
+       <origin xyz="0.05 0 0.05" rpy="${-pi/4} ${-pi/2} 0" />
+  </xacro:realsense-rs200>
+  <!--end for camera link-->
 </robot>
